File: sch/boilers/boilers.sch (EAGLE design)
At the start: 12 parts, among them IC1 74HC165N, IC2 74HCT595N, J1 22-27-2041-04

Commit message: 11
Parts:
- removed TEMP_SENSOR, TEMP_SENSOR1, TEMP_SENSOR2, TEMP_SENSOR3: 22-27-2031-03, con-molex:22-27-2031-03
- added DISPLAY: 22-27-2051-05, con-molex:22-27-2051-05
- added J2: 22-27-2081-08, con-molex:22-27-2081-08
- added J3, J4, J5, J6: 22-27-2031-03, con-molex:22-27-2031-03
Connections:
- removed net RXD: COM-2.S, U$1.RXD2
- new net 1HZ: CLOCK-3.S
- new net A: IC1A.A, J2-7.S
- new net B: IC1A.B, J2-5.S
- new net C: IC1A.C, J2-3.S
- new net CLOCK: IC1A.CLK, IC2A.SCL, U$1.7/AIN1/PCINT23
- new net D: IC1A.D, J2-1.S
- new net E: IC1A.E, J2-2.S
- new net F: IC1A.F, J2-4.S
- new net G: IC1A.G, J2-6.S
- new net H: IC1A.H, J2-8.S
- new net N$1: COM-1.S, U$1.RXD2
- new net N$3: IC2A.SCK, U$1.6/OC0A/AIN0/PCINT22
- new net N$4: DISPLAY-1.S, U$1.5/OC0B/T1/PCINT21
- new net N$5: DISPLAY-2.S, U$1.4/XCK/T0/PCINT20
- new net N$6: DISPLAY-3.S, U$1.3/INT1/OC2B/PCINT19
- net +5V: now also DISPLAY-4.S, J1-4.S, J3-2.S, J4-2.S, J5-2.S, J6-2.S; no longer J1-2.S, TEMP_SENSOR-3.S, TEMP_SENSOR1-3.S, TEMP_SENSOR2-3.S, TEMP_SENSOR3-3.S
- net BOILER: now also J1-2.S; no longer J1-4.S
- net GND: now also DISPLAY-5.S, IC1A.SER, J3-1.S, J4-1.S, J5-1.S, J6-1.S; no longer TEMP_SENSOR-1.S, TEMP_SENSOR1-1.S, TEMP_SENSOR2-1.S, TEMP_SENSOR3-1.S
- net TEMP_SENSOR: now also J3-3.S, J4-3.S, J5-3.S, J6-3.S; no longer TEMP_SENSOR-2.S, TEMP_SENSOR1-2.S, TEMP_SENSOR2-2.S, TEMP_SENSOR3-2.S
- net TXD: now also COM-2.S; no longer COM-1.S
Other:
- moved on the sheet: CLOCK-1, CLOCK-2, CLOCK-3, CLOCK-4, CLOCK-5, COM-1, COM-2, COM-3, COM-4, COM-5, IC1, IC1P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

Commit message: 11
Connections:
- net N$4 renamed LED_DATA
- net N$5 renamed LED_CS
- net N$6 renamed LED_CLOCK
Changed lines of the file:
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@@
 <wire x1="-76.2" y1="-50.8" x2="-76.2" y2="-78.74" width="0.1524" layer="91"/>
 <wire x1="-76.2" y1="-78.74" x2="-78.74" y2="-78.74" width="0.1524" layer="91"/>
+<label x="-68.58" y="-50.8" size="1.778" layer="95"/>
 </segment>
 <segment>
@@
 </segment>
 </net>
-<net name="N$4" class="0">
+<net name="LED_DATA" class="0">
 <segment>
 <pinref part="U$1" gate="G$1" pin="5/OC0B/T1/PCINT21"/>
@@
 <pinref part="DISPLAY" gate="-1" pin="S"/>
 <wire x1="-55.88" y1="-30.48" x2="-58.42" y2="-30.48" width="0.1524" layer="91"/>
+<label x="-53.34" y="-40.64" size="1.778" layer="95"/>
 </segment>
 </net>
-<net name="N$5" class="0">
+<net name="LED_CS" class="0">
 <segment>
 <pinref part="DISPLAY" gate="-2" pin="S"/>
@@
 <pinref part="U$1" gate="G$1" pin="4/XCK/T0/PCINT20"/>
 <wire x1="-53.34" y1="-38.1" x2="-40.64" y2="-38.1" width="0.1524" layer="91"/>
+<label x="-53.34" y="-38.1" size="1.778" layer="95"/>
 </segment>
 </net>
-<net name="N$6" class="0">
+<net name="LED_CLOCK" class="0">
 <segment>
 <pinref part="U$1" gate="G$1" pin="3/INT1/OC2B/PCINT19"/>
@@
 <pinref part="DISPLAY" gate="-3" pin="S"/>
 <wire x1="-50.8" y1="-20.32" x2="-58.42" y2="-20.32" width="0.1524" layer="91"/>
+<label x="-55.88" y="-20.32" size="1.778" layer="95"/>
 </segment>
 </net>
@@
 <wire x1="-40.64" y1="-45.72" x2="-78.74" y2="-45.72" width="0.1524" layer="91"/>
 <wire x1="-78.74" y1="-45.72" x2="-78.74" y2="-76.2" width="0.1524" layer="91"/>
+<label x="-71.12" y="-45.72" size="1.778" layer="95"/>
 </segment>
 <segment>

Commit message: 11
Connections:
- new net INPUT: IC1A.QH, U$1.A0/ADC0/PCINT8
- net +5V: now also U$1.VCC2
- net GND: now also U$1.GND1, U$1.GND2, U$1.GND3
Other:
- moved on the sheet: DISPLAY-1, DISPLAY-2, DISPLAY-3, DISPLAY-4, DISPLAY-5
Changed lines of the file:
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@@
 <part name="J2" library="con-molex" deviceset="22-?-08" device="27-2081"/>
 <part name="DISPLAY" library="con-molex" deviceset="22-?-05" device="27-2051"/>
-<part name="P+8" library="supply1" deviceset="+5V" device=""/>
-<part name="GND9" library="supply1" deviceset="GND" device=""/>
 <part name="J3" library="con-molex" deviceset="22-?-03" device="27-2031"/>
 <part name="J4" library="con-molex" deviceset="22-?-03" device="27-2031"/>
@@
 <instance part="J2" gate="-7" x="-154.94" y="-33.02" rot="R180"/>
 <instance part="J2" gate="-8" x="-154.94" y="-27.94" rot="R180"/>
-<instance part="DISPLAY" gate="-1" x="-60.96" y="-30.48" rot="R180"/>
-<instance part="DISPLAY" gate="-2" x="-60.96" y="-25.4" rot="R180"/>
-<instance part="DISPLAY" gate="-3" x="-60.96" y="-20.32" rot="R180"/>
-<instance part="DISPLAY" gate="-4" x="-60.96" y="-15.24" rot="R180"/>
-<instance part="DISPLAY" gate="-5" x="-60.96" y="-10.16" rot="R180"/>
-<instance part="P+8" gate="1" x="-40.64" y="-2.54"/>
-<instance part="GND9" gate="1" x="-45.72" y="-12.7"/>
+<instance part="DISPLAY" gate="-1" x="-119.38" y="-149.86" rot="R180"/>
+<instance part="DISPLAY" gate="-2" x="-119.38" y="-144.78" rot="R180"/>
+<instance part="DISPLAY" gate="-3" x="-119.38" y="-139.7" rot="R180"/>
+<instance part="DISPLAY" gate="-4" x="-119.38" y="-134.62" rot="R180"/>
+<instance part="DISPLAY" gate="-5" x="-119.38" y="-129.54" rot="R180"/>
 <instance part="J3" gate="-1" x="-157.48" y="-132.08" rot="R180"/>
 <instance part="J3" gate="-2" x="-157.48" y="-127" rot="R180"/>
@@
 </instances>
 <busses>
-<bus name="A,B,C,D,E,F,G,H,GND,+5V,BOILER,PUMP,CLOCK,TEMP_SENSOR,SDA,SCL,1HZ">
+<bus name="A,B,C,D,E,F,G,H,GND,+5V,BOILER,PUMP,CLOCK,TEMP_SENSOR,SDA,SCL,1HZ,LED_DATA,LED_CS,LED_CLOCK,INPUT">
 <segment>
 <wire x1="-134.62" y1="-63.5" x2="-134.62" y2="-25.4" width="0.762" layer="92"/>
@@
 <segment>
 <wire x1="-147.32" y1="-119.38" x2="-147.32" y2="-195.58" width="0.762" layer="92"/>
+</segment>
+<segment>
+<wire x1="-109.22" y1="-124.46" x2="-109.22" y2="-157.48" width="0.762" layer="92"/>
+</segment>
+<segment>
+<wire x1="-81.28" y1="-40.64" x2="-81.28" y2="-33.02" width="0.762" layer="92"/>
 </segment>
 </bus>
@@
 <junction x="43.18" y="-71.12"/>
 <pinref part="U$1" gate="G$1" pin="GND4"/>
-<wire x1="20.32" y1="-68.58" x2="43.18" y2="-68.58" width="0.1524" layer="91"/>
+<wire x1="20.32" y1="-68.58" x2="25.4" y2="-68.58" width="0.1524" layer="91"/>
+<wire x1="25.4" y1="-68.58" x2="43.18" y2="-68.58" width="0.1524" layer="91"/>
 <wire x1="43.18" y1="-68.58" x2="43.18" y2="-71.12" width="0.1524" layer="91"/>
 <junction x="43.18" y="-68.58"/>
+<pinref part="U$1" gate="G$1" pin="GND1"/>
+<wire x1="20.32" y1="-60.96" x2="25.4" y2="-60.96" width="0.1524" layer="91"/>
+<wire x1="25.4" y1="-60.96" x2="25.4" y2="-63.5" width="0.1524" layer="91"/>
+<pinref part="U$1" gate="G$1" pin="GND2"/>
+<wire x1="20.32" y1="-63.5" x2="25.4" y2="-63.5" width="0.1524" layer="91"/>
+<wire x1="25.4" y1="-63.5" x2="25.4" y2="-66.04" width="0.1524" layer="91"/>
+<pinref part="U$1" gate="G$1" pin="GND3"/>
+<wire x1="20.32" y1="-66.04" x2="25.4" y2="-66.04" width="0.1524" layer="91"/>
+<wire x1="25.4" y1="-66.04" x2="25.4" y2="-68.58" width="0.1524" layer="91"/>
+<junction x="25.4" y="-66.04"/>
+<junction x="25.4" y="-63.5"/>
 </segment>
 <segment>
@@
 </segment>
 <segment>
-<pinref part="DISPLAY" gate="-5" pin="S"/>
-<pinref part="GND9" gate="1" pin="GND"/>
-<wire x1="-58.42" y1="-10.16" x2="-45.72" y2="-10.16" width="0.1524" layer="91"/>
-</segment>
-<segment>
 <pinref part="CLOCK" gate="-1" pin="S"/>
 <wire x1="-162.56" y1="-111.76" x2="-147.32" y2="-111.76" width="0.1524" layer="91"/>
@@
 <wire x1="-154.94" y1="-195.58" x2="-147.32" y2="-195.58" width="0.1524" layer="91"/>
 </segment>
+<segment>
+<pinref part="DISPLAY" gate="-5" pin="S"/>
+<wire x1="-116.84" y1="-129.54" x2="-109.22" y2="-129.54" width="0.1524" layer="91"/>
+</segment>
 </net>
 <net name="+5V" class="1">
 <segment>
 <pinref part="P+2" gate="1" pin="+5V"/>
-<wire x1="27.94" y1="-55.88" x2="20.32" y2="-55.88" width="0.1524" layer="91"/>
+<wire x1="27.94" y1="-55.88" x2="25.4" y2="-55.88" width="0.1524" layer="91"/>
 <pinref part="U$1" gate="G$1" pin="VCC1"/>
+<pinref part="U$1" gate="G$1" pin="VCC2"/>
+<wire x1="25.4" y1="-55.88" x2="20.32" y2="-55.88" width="0.1524" layer="91"/>
+<wire x1="20.32" y1="-58.42" x2="25.4" y2="-58.42" width="0.1524" layer="91"/>
+<wire x1="25.4" y1="-58.42" x2="25.4" y2="-55.88" width="0.1524" layer="91"/>
+<junction x="25.4" y="-55.88"/>
 </segment>
 <segment>
@@
 </segment>
 <segment>
-<pinref part="DISPLAY" gate="-4" pin="S"/>
-<pinref part="P+8" gate="1" pin="+5V"/>
-<wire x1="-58.42" y1="-15.24" x2="-40.64" y2="-15.24" width="0.1524" layer="91"/>
-<wire x1="-40.64" y1="-15.24" x2="-40.64" y2="-5.08" width="0.1524" layer="91"/>
-</segment>
-<segment>
 <pinref part="CLOCK" gate="-2" pin="S"/>
 <wire x1="-162.56" y1="-109.22" x2="-147.32" y2="-109.22" width="0.1524" layer="91"/>
@@
 <pinref part="J6" gate="-2" pin="S"/>
 <wire x1="-154.94" y1="-190.5" x2="-147.32" y2="-190.5" width="0.1524" layer="91"/>
+</segment>
+<segment>
+<pinref part="DISPLAY" gate="-4" pin="S"/>
+<wire x1="-116.84" y1="-134.62" x2="-109.22" y2="-134.62" width="0.1524" layer="91"/>
 </segment>
 </net>
@@
 <net name="LED_DATA" class="0">
 <segment>
+<pinref part="DISPLAY" gate="-1" pin="S"/>
+<wire x1="-116.84" y1="-149.86" x2="-109.22" y2="-149.86" width="0.1524" layer="91"/>
+</segment>
+<segment>
 <pinref part="U$1" gate="G$1" pin="5/OC0B/T1/PCINT21"/>
-<wire x1="-40.64" y1="-40.64" x2="-55.88" y2="-40.64" width="0.1524" layer="91"/>
-<wire x1="-55.88" y1="-40.64" x2="-55.88" y2="-30.48" width="0.1524" layer="91"/>
-<pinref part="DISPLAY" gate="-1" pin="S"/>
-<wire x1="-55.88" y1="-30.48" x2="-58.42" y2="-30.48" width="0.1524" layer="91"/>
-<label x="-53.34" y="-40.64" size="1.778" layer="95"/>
+<wire x1="-40.64" y1="-40.64" x2="-81.28" y2="-40.64" width="0.1524" layer="91"/>
+<label x="-76.2" y="-40.64" size="1.778" layer="95"/>
 </segment>
 </net>
@@
 <segment>
 <pinref part="DISPLAY" gate="-2" pin="S"/>
-<wire x1="-58.42" y1="-25.4" x2="-53.34" y2="-25.4" width="0.1524" layer="91"/>
-<wire x1="-53.34" y1="-25.4" x2="-53.34" y2="-38.1" width="0.1524" layer="91"/>
+<wire x1="-116.84" y1="-144.78" x2="-109.22" y2="-144.78" width="0.1524" layer="91"/>
+</segment>
+<segment>
 <pinref part="U$1" gate="G$1" pin="4/XCK/T0/PCINT20"/>
-<wire x1="-53.34" y1="-38.1" x2="-40.64" y2="-38.1" width="0.1524" layer="91"/>
-<label x="-53.34" y="-38.1" size="1.778" layer="95"/>
+<wire x1="-40.64" y1="-38.1" x2="-81.28" y2="-38.1" width="0.1524" layer="91"/>
+<label x="-76.2" y="-38.1" size="1.778" layer="95"/>
 </segment>
 </net>
 <net name="LED_CLOCK" class="0">
 <segment>
+<pinref part="DISPLAY" gate="-3" pin="S"/>
+<wire x1="-116.84" y1="-139.7" x2="-109.22" y2="-139.7" width="0.1524" layer="91"/>
+</segment>
+<segment>
 <pinref part="U$1" gate="G$1" pin="3/INT1/OC2B/PCINT19"/>
-<wire x1="-40.64" y1="-35.56" x2="-50.8" y2="-35.56" width="0.1524" layer="91"/>
-<wire x1="-50.8" y1="-35.56" x2="-50.8" y2="-20.32" width="0.1524" layer="91"/>
-<pinref part="DISPLAY" gate="-3" pin="S"/>
-<wire x1="-50.8" y1="-20.32" x2="-58.42" y2="-20.32" width="0.1524" layer="91"/>
-<label x="-55.88" y="-20.32" size="1.778" layer="95"/>
+<wire x1="-40.64" y1="-35.56" x2="-81.28" y2="-35.56" width="0.1524" layer="91"/>
+<label x="-76.2" y="-35.56" size="1.778" layer="95"/>
 </segment>
 </net>
@@
 </segment>
 </net>
+<net name="INPUT" class="0">
+<segment>
+<pinref part="U$1" gate="G$1" pin="A0/ADC0/PCINT8"/>
+<wire x1="-40.64" y1="-68.58" x2="-73.66" y2="-68.58" width="0.1524" layer="91"/>
+<wire x1="-73.66" y1="-68.58" x2="-73.66" y2="-81.28" width="0.1524" layer="91"/>
+<wire x1="-73.66" y1="-81.28" x2="-78.74" y2="-81.28" width="0.1524" layer="91"/>
+</segment>
+<segment>
+<pinref part="IC1" gate="A" pin="QH"/>
+<wire x1="-93.98" y1="-33.02" x2="-81.28" y2="-33.02" width="0.1524" layer="91"/>
+</segment>
+</net>

Commit message: first
Parts:
- added C1, C2, C3: (no value), rcl:C-EU050-024X044
- added D1, D2, D3: 1N4148DO35-7, diode:1N4148DO35-7
- added IC3: 74AC14N, 74xx-eu:74AC14N
- added JP1, JP2: (no value), adafruit:PINHD-1X6
- added R1, R2, R3: (no value), rcl:R-EU_0207/10
Connections:
- net N$3 renamed OUTPUT
- new net LOAD: IC1A.SH/!LD, U$1.7/AIN1/PCINT23
- new net N$10: D2.A, IC3B.O, JP2.3
- new net N$11: D1.A, IC3A.O, JP2.2
- new net N$12: IC3A.I, IC3D.O
- new net N$13: IC3B.I, IC3E.O
- new net N$14: IC3C.I, IC3F.O
- new net N$15: D1.C, D2.C, D3.C, JP2.5
- new net N$3: C3.2, IC3F.I, JP1.4, R3.2
- new net N$4: C1.2, IC3D.I, JP1.6, R1.2
- new net N$7: C2.2, IC3E.I, JP1.5
- new net N$9: D3.A, IC3C.O, JP2.4
- net +5V: now also C1.1, C2.1, C3.1, IC3P.VCC, JP1.2, JP1.3, JP2.1
- net CLOCK: now also U$1.8/CLKO/ICP1/PCINT0; no longer U$1.7/AIN1/PCINT23
- net GND: now also IC3P.GND, JP2.6, R1.1, R2.1, R3.1
Other:
- moved on the sheet: J3-1, J3-2, J3-3, J4-1, J4-2, J4-3, J5-1, J5-2, J5-3, J6-1, J6-2, J6-3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

Commit message: On branch master
Parts:
- removed C1, C2, C3: (no value), rcl:C-EU050-024X044
- removed D1, D2, D3: 1N4148DO35-7, diode:1N4148DO35-7
- removed IC3: 74AC14N, 74xx-eu:74AC14N
- removed JP1, JP2: (no value), adafruit:PINHD-1X6
- removed R1, R2, R3: (no value), rcl:R-EU_0207/10
Connections:
- removed net N$10: D2.A, IC3B.O, JP2.3
- removed net N$11: D1.A, IC3A.O, JP2.2
- removed net N$12: IC3A.I, IC3D.O
- removed net N$13: IC3B.I, IC3E.O
- removed net N$14: IC3C.I, IC3F.O
- removed net N$15: D1.C, D2.C, D3.C, JP2.5
- removed net N$3: C3.2, IC3F.I, JP1.4, R3.2
- removed net N$4: C1.2, IC3D.I, JP1.6, R1.2
- removed net N$7: C2.2, IC3E.I, JP1.5
- removed net N$9: D3.A, IC3C.O, JP2.4
- net +5V: no longer C1.1, C2.1, C3.1, IC3P.VCC, JP1.2, JP1.3, JP2.1
- net GND: no longer IC3P.GND, JP2.6, R1.1, R2.1, R3.1

Commit message: v.1.0
Parts:
- added S1: (no value), switch-omron:10-XX
- J1: value 22-27-2041-04 -> 22-27-2101-10; device con-molex:22-27-2041-04 -> con-molex:22-27-2101-10
Connections:
- net BOILER renamed QA
- net PUMP renamed QB
- removed net CLOCK: IC1A.CLK, IC2A.SCL, U$1.8/CLKO/ICP1/PCINT0
- removed net INPUT: IC1A.QH, U$1.A0/ADC0/PCINT8
- removed net LOAD: IC1A.SH/!LD, U$1.7/AIN1/PCINT23
- removed net OUTPUT: IC2A.SCK, U$1.6/OC0A/AIN0/PCINT22
- new net EXT_CLOCK: IC1A.CLK, IC2A.SCK, U$1.7/AIN1/PCINT23
- new net EXT_CS: IC2A.RCK, U$1.8/CLKO/ICP1/PCINT0
- new net EXT_CS_IN: IC1A.SH/!LD, U$1.A0/ADC0/PCINT8
- new net EXT_DATA_IN: IC1A.QH, U$1.5/OC0B/T1/PCINT21
- new net EXT_DATA_OUT: IC2A.SER, U$1.6/OC0A/AIN0/PCINT22
- new net QC: IC2A.QC, J1-4.S
- new net QD: IC2A.QD, J1-5.S
- new net QE: IC2A.QE, J1-6.S
- new net QF: IC2A.QF, J1-7.S
- new net QG: IC2A.QG, J1-8.S
- new net QH: IC2A.QH, J1-9.S
- new net RESET: S1.P, U$1.RST/PCINT14
- net +5V: now also IC1A.INH, IC1A.SER, IC2A.SCL, J1-1.S; no longer J1-4.S
- net GND: now also IC2A.G, J1-10.S, S1.S; no longer IC1A.SER, J1-1.S
- net LED_CLOCK: now also U$1.2/INT0/PCINT18; no longer U$1.3/INT1/OC2B/PCINT19
- net LED_CS: now also U$1.3/INT1/OC2B/PCINT19; no longer U$1.4/XCK/T0/PCINT20
- net LED_DATA: now also U$1.4/XCK/T0/PCINT20; no longer U$1.5/OC0B/T1/PCINT21
Other:
- moved on the sheet: J1-1, J1-2, J1-3, J1-4

Commit message: 11
Parts:
- added LED1, LED2, LED3, LED4, LED5, LED6, LED7, LED8: (no value), led:LED5MM
- added R1, R2, R3, R4, R5, R6, R7, R8: (no value), rcl:R-EU_0207/10
Connections:
- new net N$10: LED7.C, R7.2
- new net N$11: LED8.C, R8.2
- new net N$3: LED1.C, R1.2
- new net N$4: LED2.C, R2.2
- new net N$6: LED3.C, R3.2
- new net N$7: LED4.C, R4.2
- new net N$8: LED5.C, R5.2
- new net N$9: LED6.C, R6.2
- net +5V: now also LED1.A, LED2.A, LED3.A, LED4.A, LED5.A, LED6.A, LED7.A, LED8.A
- net QA: now also R1.1
- net QB: now also R2.1
- net QC: now also R3.1
- net QD: now also R4.1
- net QE: now also R5.1
- net QF: now also R6.1
- net QG: now also R7.1
- net QH: now also R8.1

Commit message: first
Parts:
- LED1, LED2, LED3, LED4, LED5, LED6, LED7, LED8: value (none) -> АЛ307Б
- R1, R2, R3, R4, R5, R6, R7, R8: value (none) -> 510
Changed lines of the file:
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@@
 <part name="J1" library="con-molex" deviceset="22-?-10" device="27-2101"/>
 <part name="S1" library="switch-omron" deviceset="10-XX" device=""/>
-<part name="LED1" library="led" deviceset="LED" device="5MM"/>
-<part name="R1" library="rcl" deviceset="R-EU_" device="0207/10"/>
-<part name="LED2" library="led" deviceset="LED" device="5MM"/>
-<part name="R2" library="rcl" deviceset="R-EU_" device="0207/10"/>
-<part name="LED3" library="led" deviceset="LED" device="5MM"/>
-<part name="R3" library="rcl" deviceset="R-EU_" device="0207/10"/>
-<part name="LED4" library="led" deviceset="LED" device="5MM"/>
-<part name="R4" library="rcl" deviceset="R-EU_" device="0207/10"/>
-<part name="LED5" library="led" deviceset="LED" device="5MM"/>
-<part name="R5" library="rcl" deviceset="R-EU_" device="0207/10"/>
-<part name="LED6" library="led" deviceset="LED" device="5MM"/>
-<part name="R6" library="rcl" deviceset="R-EU_" device="0207/10"/>
-<part name="LED7" library="led" deviceset="LED" device="5MM"/>
-<part name="R7" library="rcl" deviceset="R-EU_" device="0207/10"/>
-<part name="LED8" library="led" deviceset="LED" device="5MM"/>
-<part name="R8" library="rcl" deviceset="R-EU_" device="0207/10"/>
+<part name="LED1" library="led" deviceset="LED" device="5MM" value="АЛ307Б"/>
+<part name="R1" library="rcl" deviceset="R-EU_" device="0207/10" value="510"/>
+<part name="LED2" library="led" deviceset="LED" device="5MM" value="АЛ307Б"/>
+<part name="R2" library="rcl" deviceset="R-EU_" device="0207/10" value="510"/>
+<part name="LED3" library="led" deviceset="LED" device="5MM" value="АЛ307Б"/>
+<part name="R3" library="rcl" deviceset="R-EU_" device="0207/10" value="510"/>
+<part name="LED4" library="led" deviceset="LED" device="5MM" value="АЛ307Б"/>
+<part name="R4" library="rcl" deviceset="R-EU_" device="0207/10" value="510"/>
+<part name="LED5" library="led" deviceset="LED" device="5MM" value="АЛ307Б"/>
+<part name="R5" library="rcl" deviceset="R-EU_" device="0207/10" value="510"/>
+<part name="LED6" library="led" deviceset="LED" device="5MM" value="АЛ307Б"/>
+<part name="R6" library="rcl" deviceset="R-EU_" device="0207/10" value="510"/>
+<part name="LED7" library="led" deviceset="LED" device="5MM" value="АЛ307Б"/>
+<part name="R7" library="rcl" deviceset="R-EU_" device="0207/10" value="510"/>
+<part name="LED8" library="led" deviceset="LED" device="5MM" value="АЛ307Б"/>
+<part name="R8" library="rcl" deviceset="R-EU_" device="0207/10" value="510"/>
 <part name="P+3" library="supply1" deviceset="+5V" device=""/>
 </parts>
@@
 </sheet>
 </sheets>
+<errors>
+</errors>
 </schematic>
 </drawing>
