File: sch/boilers/boilers.sch (EAGLE design)
At the start: 31 parts, among them IC1 74HC165N, IC2 74HCT595N, J1 22-27-2101-10, J2 22-27-2081-08, J3 22-27-2031-03, J4 22-27-2031-03, J5 22-27-2031-03, J6 22-27-2031-03

Commit message: commutator
Connections:
- net +5V: no longer IC1A.INH
- net GND: now also IC1A.INH
Changed lines of the file:
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@@
 <label x="-60.96" y="-152.4" size="1.778" layer="95"/>
+</segment>
+<segment>
+<pinref part="IC1" gate="A" pin="INH"/>
+<wire x1="-119.38" y1="-58.42" x2="-134.62" y2="-58.42" width="0.1524" layer="91"/>
+<label x="-134.62" y="-58.42" size="1.778" layer="95"/>
 </segment>
 </net>
@@
 <wire x1="-119.38" y1="-83.82" x2="-147.32" y2="-83.82" width="0.1524" layer="91"/>
 <label x="-142.24" y="-83.82" size="1.778" layer="95"/>
-</segment>
-<segment>
-<pinref part="IC1" gate="A" pin="INH"/>
-<wire x1="-119.38" y1="-58.42" x2="-134.62" y2="-58.42" width="0.1524" layer="91"/>
-<label x="-134.62" y="-58.42" size="1.778" layer="95"/>
 </segment>
 <segment>
@@
 <pinref part="R3" gate="G$1" pin="1"/>
 <wire x1="-12.7" y1="-121.92" x2="-20.32" y2="-121.92" width="0.1524" layer="91"/>
+<label x="-17.78" y="-121.92" size="1.778" layer="95"/>
 </segment>
 </net>
@@
 <pinref part="R4" gate="G$1" pin="1"/>
 <wire x1="-12.7" y1="-129.54" x2="-20.32" y2="-129.54" width="0.1524" layer="91"/>
+<label x="-17.78" y="-129.54" size="1.778" layer="95"/>
 </segment>
 </net>
@@
 <pinref part="R5" gate="G$1" pin="1"/>
 <wire x1="-12.7" y1="-137.16" x2="-20.32" y2="-137.16" width="0.1524" layer="91"/>
+<label x="-17.78" y="-137.16" size="1.778" layer="95"/>
 </segment>
 </net>
@@
 <pinref part="R6" gate="G$1" pin="1"/>
 <wire x1="-12.7" y1="-144.78" x2="-20.32" y2="-144.78" width="0.1524" layer="91"/>
+<label x="-17.78" y="-144.78" size="1.778" layer="95"/>
 </segment>
 </net>
@@
 <pinref part="R7" gate="G$1" pin="1"/>
 <wire x1="-12.7" y1="-152.4" x2="-20.32" y2="-152.4" width="0.1524" layer="91"/>
+<label x="-17.78" y="-152.4" size="1.778" layer="95"/>
 </segment>
 </net>
@@
 <pinref part="R2" gate="G$1" pin="1"/>
 <wire x1="-12.7" y1="-114.3" x2="-20.32" y2="-114.3" width="0.1524" layer="91"/>
+<label x="-17.78" y="-114.3" size="1.778" layer="95"/>
 </segment>
 </net>
@@
 <pinref part="R1" gate="G$1" pin="1"/>
 <wire x1="-12.7" y1="-106.68" x2="-20.32" y2="-106.68" width="0.1524" layer="91"/>
-</segment>
-</net>
+<label x="-17.78" y="-106.68" size="1.778" layer="95"/>
+</segment>
+</net>
