File: sch/boilers/boilers.brd (EAGLE design)
At the start: 100 x 80 mm, 14 parts, among them IC1 74HC165N, IC2 74HCT595N, J1 22-27-2041-04, J2 22-27-2081-08, J3 22-27-2031-03, J4 22-27-2031-03, J5 22-27-2031-03, J6 22-27-2031-03

Commit message: 11
Connections:
- net N$4 renamed LED_DATA
- net N$5 renamed LED_CS
- net N$6 renamed LED_CLOCK
Changed lines of the file:
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@@
 <wire x1="55.88" y1="16.51" x2="55.88" y2="16.764" width="0.508" layer="16"/>
 </signal>
-<signal name="N$4">
+<signal name="LED_DATA">
 <contactref element="U$1" pad="5"/>
 <contactref element="DISPLAY" pad="1"/>
@@
 <wire x1="54.61" y1="30.48" x2="55.88" y2="31.75" width="0.508" layer="16"/>
 </signal>
-<signal name="N$5">
+<signal name="LED_CS">
 <contactref element="DISPLAY" pad="2"/>
 <contactref element="U$1" pad="4"/>
@@
 <wire x1="52.07" y1="30.48" x2="52.07" y2="30.988" width="0.508" layer="16"/>
 </signal>
-<signal name="N$6">
+<signal name="LED_CLOCK">
 <contactref element="U$1" pad="3"/>
 <contactref element="DISPLAY" pad="3"/>

Commit message: 11
Parts:
- moved POWER 15.3 mm to (40.6, 74.9), turned to 180 degrees
Connections:
- removed net VCC2: U$1.VCC2
- new net INPUT: IC1.9, U$1.A0
- net +5V: now also U$1.VCC2
- net GND: now also U$1.GND, U$1.GND2, U$1.GND3
Routing:
- net CLOCK: track 22.6 -> 85.2 mm
- net INPUT: track 0.00 -> 53.4 mm, vias 0 -> 2
- net +5V: track 257.2 -> 224.2 mm, vias 0 -> 4
- net GND: track 253.1 -> 280.3 mm, vias 0 -> 2
- net PUMP: track 23.0 -> 15.5 mm

Commit message: first
Parts:
- added C1, C2, C3: (no value), rcl:C050-024X044
- added D1, D2, D3: 1N4148DO35-7, diode:DO35-7
- added IC3: 74AC14N, 74xx-eu:DIL14
- added JP1, JP2: (no value), adafruit:1X06
- added R1, R2, R3: (no value), rcl:0207/10
- moved J5 18.0 mm to (76.2, 19.1)
- moved J3 17.8 mm to (76.2, 36.8)
- moved J4 17.8 mm to (76.2, 27.9)
- moved J6 17.8 mm to (76.2, 11.4)
- moved POWER 11.4 mm to (40.6, 63.5)
- moved SD 11.4 mm to (59.7, 63.5)
Connections:
- net N$3 renamed OUTPUT
- new net LOAD: IC1.1, U$1.7
- new net N$10: D2.A, IC3.10, JP2.3
- new net N$11: D1.A, IC3.12, JP2.2
- new net N$12: IC3.13, IC3.2
- new net N$13: IC3.11, IC3.4
- new net N$14: IC3.6, IC3.9
- new net N$15: D1.C, D2.C, D3.C, JP2.5
- new net N$3: C3.2, IC3.5, JP1.4, R3.2
- new net N$4: C1.2, IC3.1, JP1.6, R1.2
- new net N$7: C2.2, IC3.3, JP1.5
- new net N$9: D3.A, IC3.8, JP2.4
- net +5V: now also C1.1, C2.1, C3.1, IC3.14, JP1.2, JP1.3, JP2.1
- net CLOCK: now also U$1.8; no longer U$1.7
- net GND: now also IC3.7, JP2.6, R1.1, R2.1, R3.1
Routing:
- net LOAD: track 0.00 -> 62.8 mm
- net +5V: track 224.2 -> 195.1 mm
- net GND: track 280.3 -> 260.4 mm
- net TEMP_SENSOR: track 50.8 -> 33.5 mm
- net SS: track 21.6 -> 10.2 mm
- net SCK: track 21.6 -> 10.2 mm
- net MOSI: track 21.6 -> 10.2 mm
- net MISO: track 21.6 -> 10.2 mm
- net CLOCK: track 85.2 -> 89.8 mm
- net INPUT: track 53.4 -> 52.7 mm
Other:
- board size 100 x 80 mm -> 84.8 x 102.9 mm

Commit message: On branch master
Parts:
- removed C1, C2, C3: (no value), rcl:C050-024X044
- removed D1, D2, D3: 1N4148DO35-7, diode:DO35-7
- removed IC3: 74AC14N, 74xx-eu:DIL14
- removed JP1, JP2: (no value), adafruit:1X06
- removed R1, R2, R3: (no value), rcl:0207/10
Connections:
- removed net N$10: D2.A, IC3.10, JP2.3
- removed net N$11: D1.A, IC3.12, JP2.2
- removed net N$12: IC3.13, IC3.2
- removed net N$13: IC3.11, IC3.4
- removed net N$14: IC3.6, IC3.9
- removed net N$15: D1.C, D2.C, D3.C, JP2.5
- removed net N$3: C3.2, IC3.5, JP1.4, R3.2
- removed net N$4: C1.2, IC3.1, JP1.6, R1.2
- removed net N$7: C2.2, IC3.3, JP1.5
- removed net N$9: D3.A, IC3.8, JP2.4
- net +5V: no longer C1.1, C2.1, C3.1, IC3.14, JP1.2, JP1.3, JP2.1
- net GND: no longer IC3.7, JP2.6, R1.1, R2.1, R3.1
Other:
- board size 84.8 x 102.9 mm -> 84.8 x 73.7 mm
Changed lines of the file:
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@@
 <board>
 <plain>
-<wire x1="0" y1="-29.21" x2="84.76" y2="-29.21" width="0" layer="20"/>
-<wire x1="84.76" y1="-29.21" x2="84.76" y2="73.65" width="0" layer="20"/>
+<wire x1="0" y1="0" x2="84.76" y2="0" width="0" layer="20"/>
+<wire x1="84.76" y1="0" x2="84.76" y2="73.65" width="0" layer="20"/>
 <wire x1="84.76" y1="73.65" x2="0" y2="73.65" width="0" layer="20"/>
-<wire x1="0" y1="73.65" x2="0" y2="-29.21" width="0" layer="20"/>
+<wire x1="0" y1="73.65" x2="0" y2="0" width="0" layer="20"/>
 <hole x="3.81" y="69.85" drill="0.6"/>
 <hole x="81.28" y="69.85" drill="0.6"/>
@@
 <attribute name="OC_FARNELL" value="unknown" x="76.2" y="11.43" size="1.778" layer="27" display="off"/>
 </element>
-<element name="IC3" library="74xx-eu" package="DIL14" value="74AC14N" x="20.32" y="7.62"/>
-<element name="C1" library="rcl" package="C050-024X044" value="" x="3.81" y="-16.51"/>
-<element name="C2" library="rcl" package="C050-024X044" value="" x="3.81" y="-21.59"/>
-<element name="C3" library="rcl" package="C050-024X044" value="" x="3.81" y="-26.67"/>
-<element name="R1" library="rcl" package="0207/10" value="" x="6.35" y="-31.75"/>
-<element name="R2" library="rcl" package="0207/10" value="" x="6.35" y="-36.83"/>
-<element name="R3" library="rcl" package="0207/10" value="" x="6.35" y="-41.91"/>
-<element name="D1" library="diode" package="DO35-7" value="1N4148DO35-7" x="6.35" y="-46.99"/>
-<element name="D2" library="diode" package="DO35-7" value="1N4148DO35-7" x="6.35" y="-53.34"/>
-<element name="D3" library="diode" package="DO35-7" value="1N4148DO35-7" x="6.35" y="-59.69"/>
-<element name="JP1" library="adafruit" package="1X06" value="" x="8.89" y="-67.31"/>
-<element name="JP2" library="adafruit" package="1X06" value="" x="8.89" y="-72.39"/>
 </elements>
 <signals>
@@
 <wire x1="53.34" y1="22.86" x2="54.61" y2="21.59" width="0.6096" layer="16"/>
 <wire x1="54.61" y1="21.59" x2="54.61" y2="12.7" width="0.4064" layer="16"/>
-<contactref element="IC3" pad="7"/>
-<contactref element="R2" pad="1"/>
-<contactref element="R3" pad="1"/>
-<contactref element="R1" pad="1"/>
-<contactref element="JP2" pad="6"/>
-<wire x1="1.27" y1="-41.91" x2="15.24" y2="-72.39" width="0" layer="19" extent="1-1"/>
-<wire x1="1.27" y1="-36.83" x2="1.27" y2="-41.91" width="0" layer="19" extent="1-1"/>
-<wire x1="1.27" y1="-31.75" x2="1.27" y2="-36.83" width="0" layer="19" extent="1-1"/>
-<wire x1="27.94" y1="3.81" x2="1.27" y2="-31.75" width="0" layer="19" extent="1-1"/>
-<wire x1="54.61" y1="12.7" x2="27.94" y2="3.81" width="0" layer="19" extent="16-16"/>
 </signal>
 <signal name="+5V" class="1">
@@
 <wire x1="45.72" y1="46.99" x2="57.15" y2="46.99" width="0.6096" layer="16"/>
 <wire x1="57.15" y1="46.99" x2="60.96" y2="50.8" width="0.6096" layer="16"/>
-<contactref element="C3" pad="1"/>
-<contactref element="C1" pad="1"/>
-<contactref element="C2" pad="1"/>
-<contactref element="IC3" pad="14"/>
-<contactref element="JP1" pad="3"/>
-<contactref element="JP1" pad="2"/>
-<contactref element="JP2" pad="1"/>
 <wire x1="76.2" y1="36.83" x2="76.2" y2="27.94" width="0" layer="19" extent="1-1"/>
-<wire x1="12.7" y1="11.43" x2="15.24" y2="16.51" width="0" layer="19" extent="16-16"/>
-<wire x1="1.27" y1="-16.51" x2="12.7" y2="11.43" width="0" layer="19" extent="1-1"/>
-<wire x1="1.27" y1="-21.59" x2="1.27" y2="-16.51" width="0" layer="19" extent="1-1"/>
-<wire x1="1.27" y1="-26.67" x2="1.27" y2="-21.59" width="0" layer="19" extent="1-1"/>
-<wire x1="5.08" y1="-67.31" x2="1.27" y2="-26.67" width="0" layer="19" extent="1-1"/>
-<wire x1="7.62" y1="-67.31" x2="5.08" y2="-67.31" width="0" layer="19" extent="1-1"/>
-<wire x1="2.54" y1="-72.39" x2="5.08" y2="-67.31" width="0" layer="19" extent="1-1"/>
 </signal>
 <signal name="TXD">
@@
 <wire x1="39.37" y1="36.83" x2="39.37" y2="40.64" width="0.4064" layer="16"/>
 </signal>
-<signal name="N$4">
-<contactref element="C1" pad="2"/>
-<contactref element="R1" pad="2"/>
-<contactref element="IC3" pad="1"/>
-<contactref element="JP1" pad="6"/>
-<wire x1="11.43" y1="-31.75" x2="15.24" y2="-67.31" width="0" layer="19" extent="1-1"/>
-<wire x1="6.35" y1="-16.51" x2="11.43" y2="-31.75" width="0" layer="19" extent="1-1"/>
-<wire x1="12.7" y1="3.81" x2="6.35" y2="-16.51" width="0" layer="19" extent="1-1"/>
-</signal>
-<signal name="N$7">
-<contactref element="C2" pad="2"/>
-<contactref element="IC3" pad="3"/>
-<contactref element="JP1" pad="5"/>
-<wire x1="6.35" y1="-21.59" x2="12.7" y2="-67.31" width="0" layer="19" extent="1-1"/>
-<wire x1="17.78" y1="3.81" x2="6.35" y2="-21.59" width="0" layer="19" extent="1-1"/>
-</signal>
-<signal name="N$3">
-<contactref element="C3" pad="2"/>
-<contactref element="R3" pad="2"/>
-<contactref element="IC3" pad="5"/>
-<contactref element="JP1" pad="4"/>
-<wire x1="11.43" y1="-41.91" x2="10.16" y2="-67.31" width="0" layer="19" extent="1-1"/>
-<wire x1="6.35" y1="-26.67" x2="11.43" y2="-41.91" width="0" layer="19" extent="1-1"/>
-<wire x1="22.86" y1="3.81" x2="6.35" y2="-26.67" width="0" layer="19" extent="1-1"/>
-</signal>
-<signal name="N$9">
-<contactref element="IC3" pad="8"/>
-<contactref element="D3" pad="A"/>
-<contactref element="JP2" pad="4"/>
-<wire x1="10.16" y1="-59.69" x2="10.16" y2="-72.39" width="0" layer="19" extent="1-1"/>
-<wire x1="27.94" y1="11.43" x2="10.16" y2="-59.69" width="0" layer="19" extent="1-1"/>
-</signal>
-<signal name="N$10">
-<contactref element="IC3" pad="10"/>
-<contactref element="D2" pad="A"/>
-<contactref element="JP2" pad="3"/>
-<wire x1="10.16" y1="-53.34" x2="7.62" y2="-72.39" width="0" layer="19" extent="1-1"/>
-<wire x1="22.86" y1="11.43" x2="10.16" y2="-53.34" width="0" layer="19" extent="1-1"/>
-</signal>
-<signal name="N$11">
-<contactref element="IC3" pad="12"/>
-<contactref element="D1" pad="A"/>
-<contactref element="JP2" pad="2"/>
-<wire x1="10.16" y1="-46.99" x2="5.08" y2="-72.39" width="0" layer="19" extent="1-1"/>
-<wire x1="17.78" y1="11.43" x2="10.16" y2="-46.99" width="0" layer="19" extent="1-1"/>
-</signal>
-<signal name="N$12">
-<contactref element="IC3" pad="2"/>
-<contactref element="IC3" pad="13"/>
-<wire x1="15.24" y1="3.81" x2="15.24" y2="11.43" width="0" layer="19" extent="1-1"/>
-</signal>
-<signal name="N$13">
-<contactref element="IC3" pad="4"/>
-<contactref element="IC3" pad="11"/>
-<wire x1="20.32" y1="11.43" x2="20.32" y2="3.81" width="0" layer="19" extent="1-1"/>
-</signal>
-<signal name="N$14">
-<contactref element="IC3" pad="6"/>
-<contactref element="IC3" pad="9"/>
-<wire x1="25.4" y1="3.81" x2="25.4" y2="11.43" width="0" layer="19" extent="1-1"/>
-</signal>
-<signal name="N$15">
-<contactref element="D3" pad="C"/>
-<contactref element="D2" pad="C"/>
-<contactref element="D1" pad="C"/>
-<contactref element="JP2" pad="5"/>
-<wire x1="2.54" y1="-59.69" x2="12.7" y2="-72.39" width="0" layer="19" extent="1-1"/>
-<wire x1="2.54" y1="-53.34" x2="2.54" y2="-59.69" width="0" layer="19" extent="1-1"/>
-<wire x1="2.54" y1="-46.99" x2="2.54" y2="-53.34" width="0" layer="19" extent="1-1"/>
-</signal>
 </signals>

Commit message: v.1.0
Parts:
- added S1: (no value), switch-omron:B3F-10XX
- J1: value 22-27-2041-04 -> 22-27-2101-10; device con-molex:6410-04 -> con-molex:6410-10
- moved J1 16.5 mm to (48.3, 6.35), turned to 180 degrees
- moved IC2 5.24 mm to (50.8, 17.8)
- moved DISPLAY 1.27 mm to (49.5, 31.8)
Connections:
- net BOILER renamed QA
- net PUMP renamed QB
- removed net CLOCK: IC1.2, IC2.10, U$1.8
- removed net INPUT: IC1.9, U$1.A0
- removed net LOAD: IC1.1, U$1.7
- removed net OUTPUT: IC2.11, U$1.6
- new net EXT_CLOCK: IC1.2, IC2.11, U$1.7
- new net EXT_CS: IC2.12, U$1.8
- new net EXT_CS_IN: IC1.1, U$1.A0
- new net EXT_DATA_IN: IC1.9, U$1.5
- new net EXT_DATA_OUT: IC2.14, U$1.6
- new net QC: IC2.2, J1.4
- new net QD: IC2.3, J1.5
- new net QE: IC2.4, J1.6
- new net QF: IC2.5, J1.7
- new net QG: IC2.6, J1.8
- new net QH: IC2.7, J1.9
- new net RESET: S1.3, U$1.RST, U$1.RST2
- net +5V: now also IC1.10, IC1.15, IC2.10, J1.1; no longer J1.4
- net GND: now also IC2.13, J1.10, S1.1; no longer IC1.10, J1.1
- net LED_CLOCK: now also U$1.2; no longer U$1.3
- net LED_CS: now also U$1.3; no longer U$1.4
- net LED_DATA: now also U$1.4; no longer U$1.5
Routing:
- net +5V: track 195.1 -> 312.0 mm
- net CLOCK: track 89.8 -> 0.00 mm
- net EXT_CS_IN: track 0.00 -> 73.3 mm, vias 0 -> 2
- net LOAD: track 62.8 -> 0.00 mm
- net EXT_CLOCK: track 0.00 -> 55.4 mm
- net INPUT: track 52.7 -> 0.00 mm, vias 2 -> 0
- net EXT_DATA_IN: track 0.00 -> 51.6 mm
- net EXT_CS: track 0.00 -> 31.5 mm
- net EXT_DATA_OUT: track 0.00 -> 27.2 mm, vias 0 -> 2
- net OUTPUT: track 22.6 -> 0.00 mm
- net QA: track 7.93 -> 18.8 mm
- net QE: track 0.00 -> 8.89 mm
- net RESET: track 0.00 -> 8.08 mm
- net QB: track 15.5 -> 7.62 mm
- net QH: track 0.00 -> 7.62 mm
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Other:
- board text added: "Boiler Control v.1.0"

Commit message: 11
Parts:
- added LED1, LED2, LED3, LED4, LED5, LED6, LED7, LED8: (no value), led:LED5MM
- added R1, R2, R3, R4, R5, R6, R7, R8: (no value), rcl:0207/10
Connections:
- new net N$10: LED7.K, R7.2
- new net N$11: LED8.K, R8.2
- new net N$3: LED1.K, R1.2
- new net N$4: LED2.K, R2.2
- new net N$6: LED3.K, R3.2
- new net N$7: LED4.K, R4.2
- new net N$8: LED5.K, R5.2
- new net N$9: LED6.K, R6.2
- net +5V: now also LED1.A, LED2.A, LED3.A, LED4.A, LED5.A, LED6.A, LED7.A, LED8.A
- net QA: now also R1.1
- net QB: now also R2.1
- net QC: now also R3.1
- net QD: now also R4.1
- net QE: now also R5.1
- net QF: now also R6.1
- net QG: now also R7.1
- net QH: now also R8.1
Routing:
- net +5V: track 312.0 -> 405.3 mm
- net N$11: track 0.00 -> 19.9 mm
- net N$3: track 0.00 -> 19.9 mm
- net N$10: track 0.00 -> 15.5 mm
- net N$4: track 0.00 -> 15.5 mm
- net N$6: track 0.00 -> 9.72 mm
- net N$9: track 0.00 -> 9.72 mm
- net N$8: track 0.00 -> 6.13 mm
- net N$7: track 0.00 -> 6.13 mm
- net QA: track 18.8 -> 23.9 mm
- net QH: track 7.62 -> 12.7 mm
- net QG: track 7.62 -> 12.7 mm
- net QF: track 7.62 -> 12.7 mm
- net QD: track 7.62 -> 12.7 mm
- net QC: track 7.62 -> 12.7 mm
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Other:
- board size 84.8 x 73.7 mm -> 84.8 x 99.1 mm

Commit message: first
Parts:
- LED1, LED2, LED3, LED4, LED5, LED6, LED7, LED8: value (none) -> АЛ307Б
- R1, R2, R3, R4, R5, R6, R7, R8: value (none) -> 510
Routing:
- net +5V: track 405.3 -> 408.9 mm
Other:
- board size 84.8 x 99.1 mm -> 86.7 x 99.1 mm
Changed lines of the file:
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@@
 <setting verticaltext="up"/>
 </settings>
-<grid distance="0.05" unitdist="inch" unit="inch" style="lines" multiple="1" display="yes" altdistance="0.025" altunitdist="inch" altunit="inch"/>
+<grid distance="0.025" unitdist="inch" unit="inch" style="lines" multiple="1" display="yes" altdistance="0.025" altunitdist="inch" altunit="mm"/>
 <layers>
 <layer number="1" name="Top" color="4" fill="1" visible="yes" active="yes"/>
@@
 <board>
 <plain>
-<wire x1="-1.27" y1="-25.4" x2="83.49" y2="-25.4" width="0" layer="20"/>
+<wire x1="-3.175" y1="-25.4" x2="83.49" y2="-25.4" width="0" layer="20"/>
 <wire x1="83.49" y1="-25.4" x2="83.49" y2="73.65" width="0" layer="20"/>
-<wire x1="83.49" y1="73.65" x2="-1.27" y2="73.65" width="0" layer="20"/>
-<wire x1="-1.27" y1="73.65" x2="-1.27" y2="-25.4" width="0" layer="20"/>
+<wire x1="83.49" y1="73.65" x2="-3.175" y2="73.65" width="0" layer="20"/>
+<wire x1="-3.175" y1="73.65" x2="-3.175" y2="-25.4" width="0" layer="20"/>
 <hole x="3.81" y="69.85" drill="0.6"/>
 <hole x="81.28" y="69.85" drill="0.6"/>
 <hole x="3.81" y="3.81" drill="0.6"/>
 <hole x="80.01" y="3.81" drill="0.6"/>
-<text x="31.75" y="66.04" size="1.016" layer="16" font="vector" rot="MR0">Boiler Control v.1.0</text>
+<text x="31.75" y="66.04" size="1.6764" layer="16" font="vector" ratio="10" rot="SMR0">Boiler Control v.1.0</text>
 </plain>
 <attributes>
@@
 <description language="de">&lt;b&gt;EAGLE Design Rules&lt;/b&gt;
 &lt;p&gt;
-Die Standard-Design-Rules sind so gewÃÂ¤hlt, dass sie fÃÂ¼r
+Die Standard-Design-Rules sind so gewählt, dass sie für
 die meisten Anwendungen passen. Sollte ihre Platine
 besondere Anforderungen haben, treffen Sie die erforderlichen
@@
 <attribute name="OC_FARNELL" value="176432" x="34.29" y="31.75" size="1.778" layer="27" rot="R180" display="off"/>
 </element>
-<element name="LED1" library="led" package="LED5MM" value="" x="21.59" y="-15.24" rot="R90"/>
-<element name="R1" library="rcl" package="0207/10" value="" x="39.37" y="-3.81" rot="R270"/>
-<element name="LED2" library="led" package="LED5MM" value="" x="29.21" y="-15.24" rot="R90"/>
-<element name="R2" library="rcl" package="0207/10" value="" x="41.91" y="-3.81" rot="R270"/>
-<element name="LED3" library="led" package="LED5MM" value="" x="36.83" y="-15.24" rot="R90"/>
-<element name="R3" library="rcl" package="0207/10" value="" x="44.45" y="-3.81" rot="R270"/>
-<element name="LED4" library="led" package="LED5MM" value="" x="44.45" y="-15.24" rot="R90"/>
-<element name="R4" library="rcl" package="0207/10" value="" x="46.99" y="-3.81" rot="R270"/>
-<element name="LED5" library="led" package="LED5MM" value="" x="52.07" y="-15.24" rot="R90"/>
-<element name="R5" library="rcl" package="0207/10" value="" x="49.53" y="-3.81" rot="R270"/>
-<element name="LED6" library="led" package="LED5MM" value="" x="59.69" y="-15.24" rot="R90"/>
-<element name="R6" library="rcl" package="0207/10" value="" x="52.07" y="-3.81" rot="R270"/>
-<element name="LED7" library="led" package="LED5MM" value="" x="67.31" y="-15.24" rot="R90"/>
-<element name="R7" library="rcl" package="0207/10" value="" x="54.61" y="-3.81" rot="R270"/>
-<element name="LED8" library="led" package="LED5MM" value="" x="74.93" y="-15.24" rot="R90"/>
-<element name="R8" library="rcl" package="0207/10" value="" x="57.15" y="-3.81" rot="R270"/>
+<element name="LED1" library="led" package="LED5MM" value="АЛ307Б" x="21.59" y="-15.24" rot="R90"/>
+<element name="R1" library="rcl" package="0207/10" value="510" x="39.37" y="-3.81" rot="R270"/>
+<element name="LED2" library="led" package="LED5MM" value="АЛ307Б" x="29.21" y="-15.24" rot="R90"/>
+<element name="R2" library="rcl" package="0207/10" value="510" x="41.91" y="-3.81" rot="R270"/>
+<element name="LED3" library="led" package="LED5MM" value="АЛ307Б" x="36.83" y="-15.24" rot="R90"/>
+<element name="R3" library="rcl" package="0207/10" value="510" x="44.45" y="-3.81" rot="R270"/>
+<element name="LED4" library="led" package="LED5MM" value="АЛ307Б" x="44.45" y="-15.24" rot="R90"/>
+<element name="R4" library="rcl" package="0207/10" value="510" x="46.99" y="-3.81" rot="R270"/>
+<element name="LED5" library="led" package="LED5MM" value="АЛ307Б" x="52.07" y="-15.24" rot="R90"/>
+<element name="R5" library="rcl" package="0207/10" value="510" x="49.53" y="-3.81" rot="R270"/>
+<element name="LED6" library="led" package="LED5MM" value="АЛ307Б" x="59.69" y="-15.24" rot="R90"/>
+<element name="R6" library="rcl" package="0207/10" value="510" x="52.07" y="-3.81" rot="R270"/>
+<element name="LED7" library="led" package="LED5MM" value="АЛ307Б" x="67.31" y="-15.24" rot="R90"/>
+<element name="R7" library="rcl" package="0207/10" value="510" x="54.61" y="-3.81" rot="R270"/>
+<element name="LED8" library="led" package="LED5MM" value="АЛ307Б" x="74.93" y="-15.24" rot="R90"/>
+<element name="R8" library="rcl" package="0207/10" value="510" x="57.15" y="-3.81" rot="R270"/>
 </elements>
 <signals>
@@
 <contactref element="IC1" pad="10"/>
 <contactref element="J1" pad="1"/>
-<wire x1="57.15" y1="21.59" x2="62.23" y2="21.59" width="0.6096" layer="16"/>
 <via x="62.23" y="21.59" extent="1-16" drill="0.6" shape="square"/>
-<wire x1="62.23" y1="21.59" x2="62.23" y2="17.78" width="0.4064" layer="1" style="shortdash"/>
-<via x="62.23" y="17.78" extent="1-16" drill="0.6" shape="square"/>
-<wire x1="62.23" y1="17.78" x2="62.23" y2="8.89" width="0.6096" layer="16"/>
+<wire x1="62.23" y1="21.59" x2="62.23" y2="16.51" width="0.4064" layer="1" style="shortdash"/>
+<via x="62.23" y="16.51" extent="1-16" drill="0.6" shape="square"/>
+<wire x1="62.23" y1="16.51" x2="62.23" y2="8.89" width="0.6096" layer="16"/>
 <wire x1="62.23" y1="8.89" x2="63.5" y2="7.62" width="0.6096" layer="16"/>
 <wire x1="63.5" y1="7.62" x2="74.93" y2="7.62" width="0.6096" layer="16"/>
@@
 <wire x1="15.24" y1="19.05" x2="15.24" y2="21.59" width="0.6096" layer="16"/>
 <wire x1="76.2" y1="36.83" x2="76.2" y2="27.94" width="0.4064" layer="16"/>
-<wire x1="15.24" y1="34.29" x2="13.97" y2="34.29" width="0.4064" layer="16"/>
+<wire x1="15.24" y1="34.29" x2="13.97" y2="34.29" width="0.6096" layer="16"/>
 <wire x1="36.83" y1="6.35" x2="19.05" y2="6.35" width="0.6096" layer="16"/>
 <wire x1="19.05" y1="6.35" x2="12.7" y2="6.35" width="0.6096" layer="16"/>
@@
 <contactref element="LED4" pad="A"/>
 <contactref element="LED2" pad="A"/>
-<wire x1="74.93" y1="-16.51" x2="67.31" y2="-16.51" width="0.4064" layer="16"/>
-<wire x1="67.31" y1="-16.51" x2="59.69" y2="-16.51" width="0.4064" layer="16"/>
-<wire x1="59.69" y1="-16.51" x2="52.07" y2="-16.51" width="0.4064" layer="16"/>
-<wire x1="52.07" y1="-16.51" x2="44.45" y2="-16.51" width="0.4064" layer="16"/>
-<wire x1="44.45" y1="-16.51" x2="36.83" y2="-16.51" width="0.4064" layer="16"/>
+<wire x1="74.93" y1="-16.51" x2="67.31" y2="-16.51" width="0.6096" layer="16"/>
+<wire x1="67.31" y1="-16.51" x2="59.69" y2="-16.51" width="0.6096" layer="16"/>
+<wire x1="59.69" y1="-16.51" x2="52.07" y2="-16.51" width="0.6096" layer="16"/>
+<wire x1="52.07" y1="-16.51" x2="44.45" y2="-16.51" width="0.6096" layer="16"/>
+<wire x1="44.45" y1="-16.51" x2="36.83" y2="-16.51" width="0.6096" layer="16"/>
 <wire x1="36.83" y1="-16.51" x2="29.21" y2="-16.51" width="0.4064" layer="16"/>
 <wire x1="29.21" y1="-16.51" x2="21.59" y2="-16.51" width="0.4064" layer="16"/>
-<wire x1="36.83" y1="-16.51" x2="21.59" y2="-16.51" width="0.4064" layer="16"/>
-<wire x1="21.59" y1="-16.51" x2="20.32" y2="-16.51" width="0.4064" layer="16"/>
-<wire x1="20.32" y1="-16.51" x2="19.05" y2="-15.24" width="0.4064" layer="16"/>
-<wire x1="19.05" y1="-15.24" x2="19.05" y2="6.35" width="0.4064" layer="16"/>
+<wire x1="36.83" y1="-16.51" x2="21.59" y2="-16.51" width="0.6096" layer="16"/>
+<wire x1="21.59" y1="-16.51" x2="20.32" y2="-16.51" width="0.6096" layer="16"/>
+<wire x1="20.32" y1="-16.51" x2="19.05" y2="-15.24" width="0.6096" layer="16"/>
+<wire x1="19.05" y1="-15.24" x2="19.05" y2="6.35" width="0.6096" layer="16"/>
+<wire x1="57.15" y1="21.59" x2="57.15" y2="22.86" width="0.4064" layer="16"/>
+<wire x1="57.15" y1="22.86" x2="58.42" y2="24.13" width="0.4064" layer="16"/>
+<wire x1="58.42" y1="24.13" x2="60.96" y2="24.13" width="0.4064" layer="16"/>
+<wire x1="60.96" y1="24.13" x2="62.23" y2="22.86" width="0.4064" layer="16"/>
+<wire x1="62.23" y1="22.86" x2="62.23" y2="21.59" width="0.4064" layer="16"/>
 </signal>
 <signal name="TXD">
@@
 </signal>
 </signals>
+<errors>
+</errors>
 </board>
 </drawing>
