File: sch/boilers/boilers.brd (EAGLE design)
At the start: 86.7 x 99.1 mm, 31 parts, among them IC1 74HC165N, IC2 74HCT595N, J1 22-27-2101-10, J2 22-27-2081-08, J3 22-27-2031-03, J4 22-27-2031-03, J5 22-27-2031-03, J6 22-27-2031-03

Commit message: commutator
Connections:
- net +5V: no longer IC1.15
- net GND: now also IC1.15
Routing:
- net GND: track 258.4 -> 278.0 mm, vias 2 -> 4
- net +5V: track 408.9 -> 406.3 mm
Changed lines of the file:
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@@
 <wire x1="34.29" y1="36.83" x2="34.29" y2="38.1" width="0.6096" layer="16"/>
 <wire x1="34.29" y1="38.1" x2="35.56" y2="39.37" width="0.6096" layer="16"/>
+<contactref element="IC1" pad="15"/>
+<wire x1="15.24" y1="21.59" x2="17.78" y2="21.59" width="0.6096" layer="16"/>
+<wire x1="17.78" y1="21.59" x2="19.05" y2="22.86" width="0.6096" layer="16"/>
+<via x="19.05" y="22.86" extent="1-16" drill="0.6"/>
+<wire x1="19.05" y1="22.86" x2="19.05" y2="36.195" width="0.4064" layer="1" style="shortdash"/>
+<via x="19.05" y="36.195" extent="1-16" drill="0.6"/>
+<wire x1="19.05" y1="36.195" x2="19.05" y2="38.1" width="0.6096" layer="16"/>
 </signal>
 <signal name="+5V" class="1">
@@
 <wire x1="57.15" y1="46.99" x2="60.96" y2="50.8" width="0.6096" layer="16"/>
 <contactref element="IC2" pad="10"/>
-<contactref element="IC1" pad="15"/>
 <contactref element="IC1" pad="10"/>
 <contactref element="J1" pad="1"/>
@@
 <wire x1="46.99" y1="46.99" x2="45.72" y2="46.99" width="0.6096" layer="16"/>
 <wire x1="45.72" y1="46.99" x2="45.72" y2="53.34" width="0.6096" layer="16"/>
-<wire x1="15.24" y1="19.05" x2="15.24" y2="21.59" width="0.6096" layer="16"/>
 <wire x1="76.2" y1="36.83" x2="76.2" y2="27.94" width="0.4064" layer="16"/>
 <wire x1="15.24" y1="34.29" x2="13.97" y2="34.29" width="0.6096" layer="16"/>
