File: sch/boilers/commutator.brd (EAGLE design)
At the start: 77.5 x 44.1 mm, 8 parts, among them IC1 74HC244N

Commit message: commutator
Parts:
- added C1, C2, C3, C4, C5, C6: (no value), rcl:C050-024X044
- added IC2: 74HC14N, 74xx-eu:DIL14
- added IC3: 74HC04N, 74xx-eu:DIL14
- added J1, J2: 22-27-2081-08, con-molex:6410-08
- added J3, J4: 22-27-2031-03, con-molex:6410-03
- added R1, R2, R3, R4, R5, R6: (no value), rcl:0207/15
Connections:
- new net N$1: IC2.12, IC3.13
- new net N$10: IC3.10, J1.4
- new net N$11: IC3.6, J1.5
- new net N$12: IC3.8, J1.6
- new net N$13: C1.2, IC2.9, J2.2, R1.2
- new net N$14: C2.2, IC2.11, J2.3, R2.2
- new net N$15: C3.2, IC2.5, J2.4, R3.2
- new net N$16: C4.2, IC2.13, J2.5, R4.2
- new net N$17: C5.2, IC2.3, J2.6, R5.2
- new net N$18: C6.2, IC2.1, J2.7, R6.2
- new net N$2: IC2.10, IC3.5
- new net N$20: J1.7, J3.1
- new net N$21: J1.8, J4.1
- new net N$3: IC2.8, IC3.9
- new net N$4: IC2.2, IC3.1
- new net N$5: IC2.4, IC3.3
- new net N$6: IC2.6, IC3.11
- new net N$7: IC3.2, J1.1
- new net N$8: IC3.12, J1.2
- new net N$9: IC3.4, J1.3
- net GND: now also IC2.7, IC3.7, J2.1, J3.3, J4.3, R1.1, R2.1, R3.1, R4.1, R5.1, R6.1
- net VCC: now also C1.1, C2.1, C3.1, C4.1, C5.1, C6.1, IC2.14, IC3.14, J2.8, J3.2, J4.2
Routing:
- net GND: track 156.9 -> 292.8 mm
- net VCC: track 96.9 -> 230.8 mm, vias 4 -> 8
- net N$13: track 0.00 -> 69.4 mm
- net N$14: track 0.00 -> 67.2 mm
- net N$16: track 0.00 -> 60.6 mm
- net N$15: track 0.00 -> 54.2 mm
- net N$17: track 0.00 -> 47.6 mm
- net N$18: track 0.00 -> 46.1 mm
- net N$20: track 0.00 -> 32.1 mm
- net N$6: track 0.00 -> 25.0 mm
- net N$21: track 0.00 -> 20.8 mm
- net N$7: track 0.00 -> 18.3 mm
- net N$11: track 0.00 -> 18.3 mm
- net N$9: track 0.00 -> 18.3 mm
- net N$1: track 0.00 -> 18.1 mm
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Other:
- board size 77.5 x 44.1 mm -> 77.5 x 82.2 mm

Commit message: display
Parts:
- added J5: 22-27-2051-05, con-molex:6410-05
- added U$1, U$2, U$3: 2X7SEG, arduino:2X7SEG
Connections:
- new net N$22: U$1.DOUT, U$2.DIN
- new net N$23: U$1.LOAD, U$2.CS
- new net N$24: J5.1, U$1.CLK, U$1.CLK2, U$2.CLK, U$2.CLK2, U$3.CLK, U$3.CLK2
- new net N$25: U$2.DOUT, U$3.DIN
- new net N$26: U$2.LOAD, U$3.CS
- new net N$27: J5.5, U$1.VCC, U$1.VCC2, U$2.VCC, U$2.VCC2, U$3.VCC, U$3.VCC2
- new net N$28: J5.4, U$1.GND, U$1.GND2, U$2.GND, U$2.GND2, U$3.GND, U$3.GND2
- new net N$29: J5.3, U$1.DIN
- new net N$30: J5.2, U$1.CS
