File: sch/boilers/commutator.sch (EAGLE design)
At the start: 8 parts, among them IC1 74HC244N

Commit message: commutator
Parts:
- added C1, C2, C3, C4, C5, C6: (no value), rcl:C-EU050-024X044
- added IC2: 74HC14N, 74xx-eu:74HC14N
- added IC3: 74HC04N, 74xx-eu:74HC04N
- added J1, J2: 22-27-2081-08, con-molex:22-27-2081-08
- added J3, J4: 22-27-2031-03, con-molex:22-27-2031-03
- added R1, R2, R3, R4, R5, R6: (no value), rcl:R-EU_0207/15
Connections:
- new net N$1: IC2A.O, IC3F.I
- new net N$10: IC3E.O, J1-4.S
- new net N$11: IC3C.O, J1-5.S
- new net N$12: IC3D.O, J1-6.S
- new net N$13: C1.2, IC2C.I, J2-2.S, R1.2
- new net N$14: C2.2, IC2B.I, J2-3.S, R2.2
- new net N$15: C3.2, IC2F.I, J2-4.S, R3.2
- new net N$16: C4.2, IC2A.I, J2-5.S, R4.2
- new net N$17: C5.2, IC2E.I, J2-6.S, R5.2
- new net N$18: C6.2, IC2D.I, J2-7.S, R6.2
- new net N$2: IC2B.O, IC3C.I
- new net N$20: J1-7.S, J3-1.S
- new net N$21: J1-8.S, J4-1.S
- new net N$3: IC2C.O, IC3D.I
- new net N$4: IC2D.O, IC3A.I
- new net N$5: IC2E.O, IC3B.I
- new net N$6: IC2F.O, IC3E.I
- new net N$7: IC3A.O, J1-1.S
- new net N$8: IC3F.O, J1-2.S
- new net N$9: IC3B.O, J1-3.S
- net GND: now also J2-1.S, J3-3.S, J4-3.S, R1.1, R2.1, R3.1, R4.1, R5.1, R6.1
- net VCC: now also C1.1, C2.1, C3.1, C4.1, C5.1, C6.1, J2-8.S, J3-2.S, J4-2.S
