File: sch/boilers/boilers2.brd (EAGLE design)
At the start: 88.9 x 106.3 mm, 32 parts, among them IC1 74HCT165N, IC2 74HCT595N, IC3 74HC04N, IC4 74HC14N, IC5 74HC244N, J1 22-27-2031-03

Commit message: first
Parts:
- added J2: А6-7, con-molex:6410-02
- CLOCK: value 22-27-2051-05 -> CLOCK
- COM: value 22-27-2031-03 -> COM
- DISPLAY: value 22-27-2051-05 -> DISPLAY
- INPUT: value 22-27-2081-08 -> INPUT
- INPUT2: value 22-27-2041-04 -> INPUT
- J1: value 22-27-2031-03 -> А1-3
- POWER: value 22-27-2021-02 -> POWER
- RELAY: value 22-27-2101-10 -> OUTPUT
- RESET: value 22-27-2021-02 -> RESET
- SD: value 22-27-2061-06 -> SPI
- moved J1 31.1 mm to (35.6, 33.0), turned to 0 degrees
- moved SD 5.08 mm to (21.6, 33.0)
Connections:
- net A6: now also J2.2
- net A7: now also J2.1
Routing:
- net A3: track 49.1 -> 7.62 mm, vias 4 -> 0
- net A2: track 43.5 -> 7.62 mm, vias 2 -> 0
- net +5V: track 518.6 -> 487.1 mm
- net A1: track 38.6 -> 7.62 mm, vias 2 -> 0
- net GND: track 516.6 -> 542.7 mm
- net A6: track 0.00 -> 18.7 mm
- net A7: track 0.00 -> 15.1 mm
- net SDA: track 96.6 -> 110.4 mm
- net SCL: track 92.3 -> 100.6 mm
- net N$22: track 78.3 -> 70.7 mm
- net N$23: track 79.0 -> 72.8 mm
- net EXT_DATA_OUT: track 23.4 -> 17.1 mm, vias 2 -> 0
- net N$29: track 98.6 -> 92.4 mm
- net N$30: track 99.4 -> 94.6 mm
- net N$26: track 118.9 -> 114.2 mm
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