File: sch/boilers/boilers2.brd (EAGLE design)
At the start: 88.9 x 106.3 mm, 33 parts, among them IC1 74HCT165N, IC2 74HCT595N, IC3 74HC04N, IC4 74HC14N, IC5 74HC244N, J1 А1-3, J2 А6-7

Commit message: first
Parts:
- moved TS1 1.27 mm to (73.7, 5.08)
- moved TS2 1.27 mm to (73.7, 15.2)
- moved TS3 1.27 mm to (73.7, 25.4)
- moved TS4 1.27 mm to (73.7, 35.6)
Routing:
- net TEMP_SENSOR: track 129.4 -> 123.6 mm
- net GND: track 542.7 -> 537.6 mm
- net +5V: track 487.1 -> 482.8 mm
Other:
- board size 88.9 x 106.3 mm -> 86.3 x 106.3 mm

Commit message: first
Other:
- board size 86.3 x 106.3 mm -> 101.6 x 195.2 mm
Changed lines of the file:
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@@
 <board>
 <plain>
-<wire x1="-6.35" y1="-6.35" x2="79.99" y2="-6.35" width="0" layer="20"/>
-<wire x1="79.99" y1="-6.35" x2="79.99" y2="100" width="0" layer="20"/>
-<wire x1="79.99" y1="100" x2="-6.35" y2="100" width="0" layer="20"/>
-<wire x1="-6.35" y1="100" x2="-6.35" y2="-6.35" width="0" layer="20"/>
+<wire x1="-21.59" y1="-6.35" x2="79.99" y2="-6.35" width="0" layer="20"/>
+<wire x1="79.99" y1="-6.35" x2="79.99" y2="188.9" width="0" layer="20"/>
+<wire x1="79.99" y1="188.9" x2="-21.59" y2="188.9" width="0" layer="20"/>
+<wire x1="-21.59" y1="188.9" x2="-21.59" y2="-6.35" width="0" layer="20"/>
 <dimension x1="-6.35" y1="-6.35" x2="-16.51" y2="189.23" x3="-30.48" y3="91.44" textsize="1.778" layer="47" dtype="vertical"/>
 <dimension x1="80.01" y1="-6.35" x2="-21.59" y2="-12.7" x3="29.21" y3="-11.43" textsize="1.778" layer="47" dtype="horizontal"/>
@@
 <wire x1="76.2" y1="53.34" x2="73.66" y2="53.34" width="0.8128" layer="16"/>
 <polygon width="0.8128" layer="16" isolate="0.6096" orphans="yes">
-<vertex x="-6.35" y="100.33"/>
-<vertex x="80.01" y="100.33"/>
+<vertex x="-21.59" y="189.23"/>
+<vertex x="80.01" y="189.23"/>
 <vertex x="80.01" y="-6.35"/>
-<vertex x="-6.35" y="-6.35"/>
+<vertex x="-21.59" y="-6.35"/>
 </polygon>
 <wire x1="17.75" y1="26.75" x2="5.25" y2="26.75" width="0.8128" layer="16"/>

Commit message: 2-й вариант
Parts:
- removed RELAY: OUTPUT, con-molex:6410-10
- added OUTPUT: 22-27-2061-06, con-molex:6410-06
- added POWER1: POWER, con-molex:6410-02
- added RL1, RL2: (no value), con-lsta:FE07
- added U$2, U$3: (no value), arduino:2CHAN_RELAY_5V
- added U$4, U$5: 5V_STAB, arduino:5V_STAB
- moved POWER 109.6 mm to (10.2, 184.2)
- moved INPUT2 2.54 mm to (12.7, 91.4)
Connections:
- new net N$37: POWER.2, U$4.N+
- new net N$38: RL1.7, RL2.7, U$5.OUT+
- new net N$40: POWER1.2, U$5.N+
- net +5V: now also OUTPUT.6, RL1.1, RL2.1, U$4.OUT+; no longer POWER.2, RELAY.10
- net GND: now also OUTPUT.1, POWER1.1, RL1.6, RL2.6, U$4.N-, U$4.OUT-, U$5.N-, U$5.OUT-; no longer RELAY.1
- net N$25: now also IC5.16, RL1.2, RL1.3; no longer IC5.18, RELAY.2
- net N$28: now also RL2.2, RL2.3; no longer RELAY.3
- net N$31: now also IC5.18, RL2.4, RL2.5; no longer IC5.16, RELAY.4
- net N$32: now also RL1.4, RL1.5; no longer RELAY.5
- net N$33: now also OUTPUT.2; no longer RELAY.6
- net N$34: now also OUTPUT.3; no longer RELAY.7
- net N$35: now also OUTPUT.4; no longer RELAY.8
- net N$36: now also OUTPUT.5; no longer RELAY.9
Routing:
- net GND: track 537.6 -> 768.1 mm, vias 6 -> 10
- net +5V: track 482.8 -> 574.2 mm, vias 7 -> 8
- net N$38: track 0.00 -> 85.9 mm
- net N$40: track 0.00 -> 85.5 mm
- net N$32: track 17.6 -> 98.8 mm
- net N$25: track 9.94 -> 82.6 mm
- net N$31: track 9.94 -> 36.6 mm
- net N$28: track 17.6 -> 35.9 mm
- net N$37: track 0.00 -> 11.4 mm
- net N$24: track 8.89 -> 6.35 mm
- net N$15: track 8.89 -> 6.35 mm
- net SDA: track 110.4 -> 111.7 mm
Other:
- board size 101.6 x 195.2 mm -> 88.9 x 195.2 mm

Commit message: 123
Parts:
- added U$6: HC-11, arduino:HC-11
- J1: value А1-3 -> 22-27-2021-02; device con-molex:6410-03 -> con-molex:6410-02
- J2: value А6-7 -> 22-27-2021-02
- moved J1 5.33 mm to (40.9, 33.0)
- moved SD 2.54 mm to (24.1, 33.0)
- moved J2 1.27 mm to (8.89, 33.0)
Connections:
- net +5V: now also J1.1, U$6.SET, U$6.VCC
- net A1: now also U$6.TXD; no longer J1.3
- net A2: now also U$6.RXD; no longer J1.2
- net A3: now also J1.2; no longer J1.1
- net GND: now also U$6.GND
Routing:
- net A1: track 7.62 -> 48.9 mm, vias 0 -> 2
- net A2: track 7.62 -> 44.5 mm, vias 0 -> 2
- net +5V: track 574.2 -> 608.2 mm
- net GND: track 768.1 -> 784.9 mm
- net SCL: track 100.6 -> 98.7 mm
- net SDA: track 111.7 -> 113.3 mm
- net SS: track 9.72 -> 8.22 mm
- net SCK: track 9.72 -> 8.22 mm
- net MOSI: track 9.72 -> 8.22 mm
- net MISO: track 9.72 -> 8.22 mm
- net N$39: track 23.4 -> 21.9 mm
- net A3: track 7.62 -> 8.25 mm
- net A6: track 18.7 -> 19.2 mm
- net A7: track 15.1 -> 15.6 mm
