File: sch/boilers/boilers2.sch (EAGLE design)
At the start: 32 parts, among them IC1 74HCT165N, IC2 74HCT595N, IC3 74HC04N, IC4 74HC14N, IC5 74HC244N, J1 22-27-2031-03

Commit message: first
Parts:
- added J2: А6-7, con-molex:22-27-2021-02
- CLOCK: value 22-27-2051-05 -> CLOCK
- COM: value 22-27-2031-03 -> COM
- DISPLAY: value 22-27-2051-05 -> DISPLAY
- INPUT: value 22-27-2081-08 -> INPUT
- INPUT2: value 22-27-2041-04 -> INPUT
- J1: value 22-27-2031-03 -> А1-3
- POWER: value 22-27-2021-02 -> POWER
- RELAY: value 22-27-2101-10 -> OUTPUT
- RESET: value 22-27-2021-02 -> RESET
- SD: value 22-27-2061-06 -> SPI
Connections:
- net A6: now also J2-2.S
- net A7: now also J2-1.S
Changed lines of the file:
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@@
 <part name="P+5" library="supply1" deviceset="+5V" device=""/>
 <part name="GND6" library="supply1" deviceset="GND" device=""/>
-<part name="RELAY" library="con-molex" deviceset="22-?-10" device="27-2101"/>
+<part name="RELAY" library="con-molex" deviceset="22-?-10" device="27-2101" value="OUTPUT"/>
 <part name="P+6" library="supply1" deviceset="+5V" device=""/>
 <part name="GND7" library="supply1" deviceset="GND" device=""/>
-<part name="DISPLAY" library="con-molex" deviceset="22-?-05" device="27-2051"/>
-<part name="CLOCK" library="con-molex" deviceset="22-?-05" device="27-2051"/>
-<part name="SD" library="con-molex" deviceset="22-?-06" device="27-2061"/>
-<part name="INPUT" library="con-molex" deviceset="22-?-08" device="27-2081"/>
-<part name="INPUT2" library="con-molex" deviceset="22-?-04" device="27-2041"/>
-<part name="COM" library="con-molex" deviceset="22-?-03" device="27-2031"/>
-<part name="RESET" library="con-molex" deviceset="22-?-02" device="27-2021"/>
-<part name="POWER" library="con-molex" deviceset="22-?-02" device="27-2021"/>
+<part name="DISPLAY" library="con-molex" deviceset="22-?-05" device="27-2051" value="DISPLAY"/>
+<part name="CLOCK" library="con-molex" deviceset="22-?-05" device="27-2051" value="CLOCK"/>
+<part name="SD" library="con-molex" deviceset="22-?-06" device="27-2061" value="SPI"/>
+<part name="INPUT" library="con-molex" deviceset="22-?-08" device="27-2081" value="INPUT"/>
+<part name="INPUT2" library="con-molex" deviceset="22-?-04" device="27-2041" value="INPUT"/>
+<part name="COM" library="con-molex" deviceset="22-?-03" device="27-2031" value="COM"/>
+<part name="RESET" library="con-molex" deviceset="22-?-02" device="27-2021" value="RESET"/>
+<part name="POWER" library="con-molex" deviceset="22-?-02" device="27-2021" value="POWER"/>
 <part name="P+9" library="supply1" deviceset="+5V" device=""/>
 <part name="GND10" library="supply1" deviceset="GND" device=""/>
-<part name="J1" library="con-molex" deviceset="22-?-03" device="27-2031"/>
+<part name="J1" library="con-molex" deviceset="22-?-03" device="27-2031" value="А1-3"/>
 <part name="TS4" library="con-molex" deviceset="22-?-03" device="05-7038"/>
 <part name="TS3" library="con-molex" deviceset="22-?-03" device="05-7038"/>
@@
 <part name="TS1" library="con-molex" deviceset="22-?-03" device="05-7038"/>
 <part name="GND8" library="supply1" deviceset="GND" device=""/>
+<part name="J2" library="con-molex" deviceset="22-?-02" device="27-2021" value="А6-7"/>
 </parts>
 <sheets>
@@
 <instance part="TS1" gate="-3" x="96.52" y="170.18" rot="R180"/>
 <instance part="GND8" gate="1" x="124.46" y="218.44"/>
+<instance part="J2" gate="-1" x="182.88" y="91.44"/>
+<instance part="J2" gate="-2" x="182.88" y="86.36"/>
 </instances>
 <busses>
@@
 <label x="170.18" y="119.38" size="1.778" layer="95"/>
 </segment>
+<segment>
+<pinref part="J2" gate="-2" pin="S"/>
+<wire x1="180.34" y1="86.36" x2="165.1" y2="86.36" width="0.1524" layer="91"/>
+</segment>
 </net>
 <net name="A7" class="0">
@@
 <label x="170.18" y="116.84" size="1.778" layer="95"/>
 </segment>
-</net>
+<segment>
+<pinref part="J2" gate="-1" pin="S"/>
+<wire x1="180.34" y1="91.44" x2="165.1" y2="91.44" width="0.1524" layer="91"/>
+</segment>
+</net>

Commit message: 2-й вариант
Parts:
- removed RELAY: OUTPUT, con-molex:22-27-2101-10
- added OUTPUT: 22-27-2061-06, con-molex:22-27-2061-06
- added POWER1: POWER, con-molex:22-27-2021-02
- added RL1, RL2: (no value), con-lsta:FE07-1
- added U$4, U$5: 5V_STAB, arduino:5V_STAB
Connections:
- new net N$37: POWER-2.S, U$4.N+
- new net N$38: RL1.7, RL2.7, U$5.OUT+
- new net N$40: POWER1-2.S, U$5.N+
- net +5V: now also OUTPUT-6.S, RL1.1, RL2.1, U$4.OUT+; no longer POWER-2.S, RELAY-10.S
- net GND: now also OUTPUT-1.S, POWER1-1.S, RL1.6, RL2.6, U$4.N-, U$4.OUT-, U$5.N-, U$5.OUT-; no longer RELAY-1.S
- net N$25: now also IC5A.Y2, RL1.2, RL1.3; no longer IC5A.Y1, RELAY-2.S
- net N$28: now also RL2.2, RL2.3; no longer RELAY-3.S
- net N$31: now also IC5A.Y1, RL2.4, RL2.5; no longer IC5A.Y2, RELAY-4.S
- net N$32: now also RL1.4, RL1.5; no longer RELAY-5.S
- net N$33: now also OUTPUT-2.S; no longer RELAY-6.S
- net N$34: now also OUTPUT-3.S; no longer RELAY-7.S
- net N$35: now also OUTPUT-4.S; no longer RELAY-8.S
- net N$36: now also OUTPUT-5.S; no longer RELAY-9.S
Other:
- moved on the sheet: INPUT-1, INPUT-2, INPUT-3, INPUT-4, INPUT-5, INPUT-6, INPUT-7, INPUT-8

Commit message: 123
Parts:
- added U$6: HC-11, arduino:HC-11
- J1: value А1-3 -> 22-27-2021-02; device con-molex:22-27-2031-03 -> con-molex:22-27-2021-02
- J2: value А6-7 -> 22-27-2021-02
Connections:
- net +5V: now also J1-1.S, U$6.SET, U$6.VCC
- net A1: now also U$6.TXD; no longer J1-3.S
- net A2: now also U$6.RXD; no longer J1-2.S
- net A3: now also J1-2.S; no longer J1-1.S
- net GND: now also U$6.GND
Other:
- moved on the sheet: J1-1, J1-2, J2-1, J2-2
Changed lines of the file:
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@@
 <part name="P+9" library="supply1" deviceset="+5V" device=""/>
 <part name="GND10" library="supply1" deviceset="GND" device=""/>
-<part name="J1" library="con-molex" deviceset="22-?-03" device="27-2031" value="А1-3"/>
 <part name="TS4" library="con-molex" deviceset="22-?-03" device="05-7038"/>
 <part name="TS3" library="con-molex" deviceset="22-?-03" device="05-7038"/>
@@
 <part name="TS1" library="con-molex" deviceset="22-?-03" device="05-7038"/>
 <part name="GND8" library="supply1" deviceset="GND" device=""/>
-<part name="J2" library="con-molex" deviceset="22-?-02" device="27-2021" value="А6-7"/>
 <part name="U$4" library="arduino" deviceset="5V_STAB" device=""/>
 <part name="U$5" library="arduino" deviceset="5V_STAB" device=""/>
@@
 <part name="RL1" library="con-lsta" deviceset="FE07-1" device=""/>
 <part name="RL2" library="con-lsta" deviceset="FE07-1" device=""/>
+<part name="U$6" library="arduino" deviceset="HC-11" device=""/>
+<part name="P+7" library="supply1" deviceset="+5V" device=""/>
+<part name="J2" library="con-molex" deviceset="22-?-02" device="27-2021"/>
+<part name="J1" library="con-molex" deviceset="22-?-02" device="27-2021"/>
 </parts>
 <sheets>
@@
 <instance part="R6" gate="G$1" x="25.4" y="185.42" rot="R90"/>
 <instance part="P+5" gate="1" x="271.78" y="154.94"/>
-<instance part="GND6" gate="1" x="274.32" y="116.84"/>
+<instance part="GND6" gate="1" x="274.32" y="63.5"/>
 <instance part="P+6" gate="1" x="322.58" y="205.74" rot="R270"/>
 <instance part="GND7" gate="1" x="309.88" y="241.3"/>
@@
 <instance part="P+9" gate="1" x="195.58" y="322.58"/>
 <instance part="GND10" gate="1" x="177.8" y="289.56"/>
-<instance part="J1" gate="-1" x="182.88" y="111.76"/>
-<instance part="J1" gate="-2" x="182.88" y="106.68"/>
-<instance part="J1" gate="-3" x="182.88" y="101.6"/>
 <instance part="TS4" gate="-1" x="96.52" y="106.68" rot="R180"/>
 <instance part="TS4" gate="-2" x="96.52" y="111.76" rot="R180"/>
@@
 <instance part="TS1" gate="-3" x="96.52" y="170.18" rot="R180"/>
 <instance part="GND8" gate="1" x="124.46" y="218.44"/>
-<instance part="J2" gate="-1" x="182.88" y="91.44"/>
-<instance part="J2" gate="-2" x="182.88" y="86.36"/>
 <instance part="U$4" gate="G$1" x="177.8" y="302.26"/>
 <instance part="U$5" gate="G$1" x="177.8" y="276.86"/>
@@
 <instance part="RL1" gate="G$1" x="332.74" y="309.88" rot="R180"/>
 <instance part="RL2" gate="G$1" x="332.74" y="281.94" rot="R180"/>
+<instance part="U$6" gate="G$1" x="243.84" y="93.98"/>
+<instance part="P+7" gate="1" x="208.28" y="78.74" rot="R90"/>
+<instance part="J2" gate="-1" x="185.42" y="91.44"/>
+<instance part="J2" gate="-2" x="185.42" y="86.36"/>
+<instance part="J1" gate="-1" x="185.42" y="78.74"/>
+<instance part="J1" gate="-2" x="185.42" y="73.66"/>
 </instances>
 <busses>
 <bus name="A,B,C,D,E,F,G,H,GND,+5V,BOILER,PUMP,EXT_CLOCK,TEMP_SENSOR,SDA,SCL,1HZ,LED_DATA,LED_CS,LED_CLOCK,SS,MOSI,MISO,SCK,EXT_DATA_OUT,LOAD,EXT_CS_IN,EXT_CS,EXT_DATA_IN,A1,A2,A3,A6,A7">
 <segment>
-<wire x1="165.1" y1="172.72" x2="165.1" y2="81.28" width="0.762" layer="92"/>
+<wire x1="165.1" y1="172.72" x2="165.1" y2="66.04" width="0.762" layer="92"/>
 </segment>
 <segment>
@@
 <wire x1="312.42" y1="289.56" x2="325.12" y2="289.56" width="0.1524" layer="91"/>
 </segment>
+<segment>
+<pinref part="P+7" gate="1" pin="+5V"/>
+<pinref part="U$6" gate="G$1" pin="VCC"/>
+<wire x1="210.82" y1="78.74" x2="215.9" y2="78.74" width="0.1524" layer="91"/>
+<pinref part="U$6" gate="G$1" pin="SET"/>
+<wire x1="215.9" y1="78.74" x2="228.6" y2="78.74" width="0.1524" layer="91"/>
+<wire x1="228.6" y1="99.06" x2="215.9" y2="99.06" width="0.1524" layer="91"/>
+<wire x1="215.9" y1="99.06" x2="215.9" y2="78.74" width="0.1524" layer="91"/>
+<junction x="215.9" y="78.74"/>
+</segment>
+<segment>
+<pinref part="J1" gate="-1" pin="S"/>
+<wire x1="182.88" y1="78.74" x2="165.1" y2="78.74" width="0.1524" layer="91"/>
+</segment>
 </net>
 <net name="GND" class="0">
@@
 <wire x1="274.32" y1="134.62" x2="274.32" y2="132.08" width="0.1524" layer="91"/>
 <pinref part="U$1" gate="G$1" pin="GND4"/>
-<wire x1="274.32" y1="132.08" x2="274.32" y2="119.38" width="0.1524" layer="91"/>
+<wire x1="274.32" y1="132.08" x2="274.32" y2="106.68" width="0.1524" layer="91"/>
+<wire x1="274.32" y1="106.68" x2="274.32" y2="66.04" width="0.1524" layer="91"/>
 <wire x1="259.08" y1="134.62" x2="274.32" y2="134.62" width="0.1524" layer="91"/>
 <pinref part="COM" gate="-1" pin="S"/>
@@
 <label x="264.16" y="137.16" size="1.778" layer="95"/>
 <label x="264.16" y="134.62" size="1.778" layer="95"/>
+<pinref part="U$6" gate="G$1" pin="GND"/>
+<wire x1="228.6" y1="83.82" x2="220.98" y2="83.82" width="0.1524" layer="91"/>
+<wire x1="220.98" y1="83.82" x2="220.98" y2="106.68" width="0.1524" layer="91"/>
+<wire x1="220.98" y1="106.68" x2="274.32" y2="106.68" width="0.1524" layer="91"/>
+<junction x="274.32" y="106.68"/>
 </segment>
 <segment>
@@
 </segment>
 <segment>
-<pinref part="J1" gate="-3" pin="S"/>
-<wire x1="180.34" y1="101.6" x2="165.1" y2="101.6" width="0.1524" layer="91"/>
-<label x="170.18" y="101.6" size="1.778" layer="95"/>
+<wire x1="165.1" y1="106.68" x2="210.82" y2="106.68" width="0.1524" layer="91"/>
+<wire x1="210.82" y1="106.68" x2="210.82" y2="93.98" width="0.1524" layer="91"/>
+<pinref part="U$6" gate="G$1" pin="TXD"/>
+<wire x1="210.82" y1="93.98" x2="228.6" y2="93.98" width="0.1524" layer="91"/>
+<label x="170.18" y="106.68" size="1.778" layer="95"/>
 </segment>
 </net>
@@
 </segment>
 <segment>
-<pinref part="J1" gate="-2" pin="S"/>
-<wire x1="180.34" y1="106.68" x2="165.1" y2="106.68" width="0.1524" layer="91"/>
-<label x="170.18" y="106.68" size="1.778" layer="95"/>
+<wire x1="165.1" y1="101.6" x2="205.74" y2="101.6" width="0.1524" layer="91"/>
+<wire x1="205.74" y1="101.6" x2="205.74" y2="88.9" width="0.1524" layer="91"/>
+<pinref part="U$6" gate="G$1" pin="RXD"/>
+<wire x1="205.74" y1="88.9" x2="228.6" y2="88.9" width="0.1524" layer="91"/>
+<label x="170.18" y="101.6" size="1.778" layer="95"/>
 </segment>
 </net>
@@
 </segment>
 <segment>
-<pinref part="J1" gate="-1" pin="S"/>
-<wire x1="180.34" y1="111.76" x2="165.1" y2="111.76" width="0.1524" layer="91"/>
-<label x="170.18" y="111.76" size="1.778" layer="95"/>
+<pinref part="J1" gate="-2" pin="S"/>
+<wire x1="182.88" y1="73.66" x2="165.1" y2="73.66" width="0.1524" layer="91"/>
 </segment>
 </net>
@@
 </segment>
 <segment>
+<wire x1="182.88" y1="86.36" x2="165.1" y2="86.36" width="0.1524" layer="91"/>
+<label x="167.64" y="86.36" size="1.778" layer="95"/>
 <pinref part="J2" gate="-2" pin="S"/>
-<wire x1="180.34" y1="86.36" x2="165.1" y2="86.36" width="0.1524" layer="91"/>
 </segment>
 </net>
@@
 </segment>
 <segment>
+<wire x1="182.88" y1="91.44" x2="165.1" y2="91.44" width="0.1524" layer="91"/>
+<label x="167.64" y="91.44" size="1.778" layer="95"/>
 <pinref part="J2" gate="-1" pin="S"/>
-<wire x1="180.34" y1="91.44" x2="165.1" y2="91.44" width="0.1524" layer="91"/>
-</segment>
-</net>
+</segment>
+</net>
