File: sch/street_lamp_controller/street_lamp_controller.brd (EAGLE design)
At the start: 43.2 x 35.2 mm, 8 parts, among them IC1 TINY15LP, J1 22-27-2031-03, J2 22-27-2021-02

Commit message: дополнительный выход
Parts:
- added J3: 22-27-2031-03, con-molex:6410-03
- moved J2 19.0 mm to (35.6, 77.5), turned to 90 degrees
Connections:
- new net N$6: IC1.1, J3.3
- net +5V: now also J2.1, J3.2; no longer J2.2
- net GND: now also J2.2, J3.1; no longer J2.1
Routing:
- net N$6: track 0.00 -> 86.8 mm
- net +5V: track 107.1 -> 115.0 mm
- net GND: track 84.8 -> 89.4 mm
Other:
- board size 43.2 x 35.2 mm -> 45.7 x 37.8 mm
