File: sch/street_lamp_controller/street_lamp_controller.sch (EAGLE design)
At the start: 8 parts, among them IC1 TINY15LP, J1 22-27-2031-03, J2 22-27-2021-02

Commit message: дополнительный выход
Parts:
- added J3: 22-27-2031-03, con-molex:22-27-2031-03
Connections:
- new net N$6: IC1.(ADC0)PB5, J3-3.S
- net +5V: now also J2-1.S, J3-2.S; no longer J2-2.S
- net GND: now also J2-2.S, J3-1.S; no longer J2-1.S
Changed lines of the file:
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@@
 <part name="SV1" library="con-lsta" deviceset="FE07-1" device=""/>
 <part name="J2" library="con-molex" deviceset="22-?-02" device="27-2021"/>
+<part name="J3" library="con-molex" deviceset="22-?-03" device="27-2031"/>
 </parts>
 <sheets>
@@
 <instance part="J2" gate="-1" x="66.04" y="40.64"/>
 <instance part="J2" gate="-2" x="66.04" y="35.56"/>
+<instance part="J3" gate="-1" x="66.04" y="27.94"/>
+<instance part="J3" gate="-2" x="66.04" y="22.86"/>
+<instance part="J3" gate="-3" x="66.04" y="17.78"/>
 </instances>
 <busses>
@@
 <wire x1="60.96" y1="104.14" x2="53.34" y2="104.14" width="0.1524" layer="91"/>
 <wire x1="53.34" y1="104.14" x2="53.34" y2="58.42" width="0.1524" layer="91"/>
-<pinref part="J2" gate="-1" pin="S"/>
-<wire x1="63.5" y1="40.64" x2="40.64" y2="40.64" width="0.1524" layer="91"/>
-<wire x1="40.64" y1="40.64" x2="40.64" y2="58.42" width="0.1524" layer="91"/>
+<wire x1="40.64" y1="35.56" x2="40.64" y2="58.42" width="0.1524" layer="91"/>
 <junction x="40.64" y="58.42"/>
+<pinref part="J3" gate="-1" pin="S"/>
+<wire x1="63.5" y1="27.94" x2="53.34" y2="27.94" width="0.1524" layer="91"/>
+<wire x1="53.34" y1="27.94" x2="53.34" y2="58.42" width="0.1524" layer="91"/>
+<pinref part="J2" gate="-2" pin="S"/>
+<wire x1="40.64" y1="35.56" x2="63.5" y2="35.56" width="0.1524" layer="91"/>
 </segment>
 </net>
@@
 <pinref part="SV1" gate="G$1" pin="6"/>
 <wire x1="60.96" y1="106.68" x2="50.8" y2="106.68" width="0.1524" layer="91"/>
-<wire x1="50.8" y1="53.34" x2="50.8" y2="35.56" width="0.1524" layer="91"/>
-<pinref part="J2" gate="-2" pin="S"/>
-<wire x1="50.8" y1="35.56" x2="63.5" y2="35.56" width="0.1524" layer="91"/>
+<wire x1="50.8" y1="53.34" x2="50.8" y2="40.64" width="0.1524" layer="91"/>
 <junction x="50.8" y="53.34"/>
+<pinref part="J3" gate="-2" pin="S"/>
+<wire x1="50.8" y1="40.64" x2="50.8" y2="22.86" width="0.1524" layer="91"/>
+<wire x1="63.5" y1="22.86" x2="50.8" y2="22.86" width="0.1524" layer="91"/>
+<pinref part="J2" gate="-1" pin="S"/>
+<wire x1="63.5" y1="40.64" x2="50.8" y2="40.64" width="0.1524" layer="91"/>
+<junction x="50.8" y="40.64"/>
 </segment>
 </net>
@@
 </segment>
 </net>
+<net name="N$6" class="0">
+<segment>
+<pinref part="J3" gate="-3" pin="S"/>
+<wire x1="63.5" y1="17.78" x2="27.94" y2="17.78" width="0.1524" layer="91"/>
+<wire x1="27.94" y1="17.78" x2="27.94" y2="81.28" width="0.1524" layer="91"/>
+<pinref part="IC1" gate="G$1" pin="(ADC0)PB5"/>
+<wire x1="27.94" y1="81.28" x2="25.4" y2="81.28" width="0.1524" layer="91"/>
+</segment>
+</net>
